Commit message: Add files via upload

File: Simple_Autonomous/robot_description.urdf.xacro (robot description, xacro)
@@ -58,5 +58,5 @@
         <child link="zed_front_camera_link"/>
         <!-- TODO: set to your actual mount position -->
-        <origin xyz="0.30 0.00 0.40" rpy="0 0 0"/>
+        <origin xyz="0.450 0.00 0.680" rpy="0 0 0"/>
     </joint>
     <!-- Front Left Wheel Link -->
