Commit message: add Camera/marvinv2.py and update Camera/new_camera_gui.py add IK_code/# two_link_plotter.py and update IK_code/armik.py add point_nav/config/goal_inputs.defaults.yaml and move/tune defaults in nav configs update EKF fusion settings and launch wiring in point_nav.launch.py extend set_goal_cli.py options/behavior and align with config-driven params add helper scripts: tools/setup_ws.sh and tools/Launch Zed Cameras.sh update rover URDF and robot_description.urdf.xacro refresh README, QUICKSTART, MOVING, and TODO with the new workflow

File: point_nav/urdf/point_nav_rover.urdf (robot description, URDF)
Before this commit: robot point_nav_rover, 8 links, 7 joints
Links:
- added link zed_left_camera_link
- added link zed_right_camera_link
Joints:
- added joint zed_left_mount_joint: type fixed, parent base_link, child zed_left_camera_link, origin xyz=0.3095 0.30232 0.21478 rpy=0 -0.523599 1.5708
- added joint zed_right_mount_joint: type fixed, parent base_link, child zed_right_camera_link, origin xyz=0.3095 -0.30232 0.21478 rpy=0 -0.523599 -1.5708
- joint zed_front_mount_joint: origin xyz=0.45 0.00 0.68 rpy=0 0 0 -> xyz=0.319521 0.0 0.342128 rpy=0 -0.523599 0

File: point_nav/urdf/robot_description.urdf.xacro (robot description, xacro)
@@ -1,4 +1,8 @@
 <?xml version="1.0"?>
 <robot xmlns:xacro="http://www.ros.org/wiki/xacro" name="robot">
+    <!-- Camera model args let you swap zed2i/zedm/other supported models without editing joints -->
+    <xacro:arg name="camera_model_front" default="zed2i" />
+    <xacro:arg name="camera_model_left" default="zed2i" />
+    <xacro:arg name="camera_model_right" default="zed2i" />
     <xacro:include filename="inertial_macros.xacro" />
     <!-- ZED include (needed for xacro:zed_camera) -->
@@ -49,5 +53,5 @@
     </gazebo>
     <!-- ZED 2i camera instance (minimal) -->
-    <xacro:zed_camera name="zed_front" model="zed2i">
+    <xacro:zed_camera name="zed_front" model="$(arg camera_model_front)">
         <!-- Required block to avoid "Not enough blocks" -->
         <gnss_origin />
@@ -57,12 +61,9 @@
         <parent link="base_link"/>
         <child link="zed_front_camera_link"/>
-        <!-- TODO: set to your actual mount position -->
-        <origin xyz="0.450 0.00 0.680" rpy="0 0 0"/>
+        <!-- From box geometry: x=0.385-0.065479, y=0, z=0.125+0.217128; 30 deg incline -->
+        <origin xyz="0.319521 0.0 0.342128" rpy="0 -0.523599 0"/>
     </joint>
-    <!-- ------------------------------------------------------------------ -->
-    <!-- PLACEHOLDERS FOR FUTURE CAMERAS (disabled/commented by default)    -->
-    <!-- Keep commented until hardware and launch topics are ready.          -->
-    <!--
-    <xacro:zed_camera name="zed_left" model="zed2i">
+    <!-- Additional side cameras -->
+    <xacro:zed_camera name="zed_left" model="$(arg camera_model_left)">
         <gnss_origin />
     </xacro:zed_camera>
@@ -70,7 +71,7 @@
         <parent link="base_link"/>
         <child link="zed_left_camera_link"/>
-        <origin xyz="0.10 0.30 0.68" rpy="0 0 1.5708"/>
+        <origin xyz="0.3095 0.30232 0.21478" rpy="0 -0.523599 1.5708"/>
     </joint>
-    <xacro:zed_camera name="zed_right" model="zed2i">
+    <xacro:zed_camera name="zed_right" model="$(arg camera_model_right)">
         <gnss_origin />
     </xacro:zed_camera>
@@ -78,7 +79,6 @@
         <parent link="base_link"/>
         <child link="zed_right_camera_link"/>
-        <origin xyz="0.10 -0.30 0.68" rpy="0 0 -1.5708"/>
+        <origin xyz="0.3095 -0.30232 0.21478" rpy="0 -0.523599 -1.5708"/>
     </joint>
-    -->
     <!-- Front Left Wheel Link -->
     <joint name="front_left_wheel_joint" type="continuous">

Commit message: Move and expand the mast Teensy sketch with raise/lower/stow serial commands Add mast operating instructions for serial control and debugging Add a simple ethernet throughput measurement note Comment out the front ZED camera odometry input in EKF fusion config Comment out the front ZED camera mount in the plain URDF Comment out the front ZED camera instance and mount in the xacro Remove the older duplicate mast sketch from its previous location

File: point_nav/urdf/point_nav_rover.urdf (robot description, URDF)
Before this commit: robot point_nav_rover, 10 links, 9 joints
Links:
- removed link zed_front_camera_link
Joints:
- removed joint zed_front_mount_joint

File: point_nav/urdf/robot_description.urdf.xacro (robot description, xacro)
@@ -52,16 +52,17 @@
         <material>Gazebo/Blue</material>
     </gazebo>
-    <!-- ZED 2i camera instance (minimal) -->
+    <!-- ZED 2i camera instance (minimal)
     <xacro:zed_camera name="zed_front" model="$(arg camera_model_front)">
-        <!-- Required block to avoid "Not enough blocks" -->
+        Required block to avoid "Not enough blocks"
         <gnss_origin />
     </xacro:zed_camera>
-    <!-- Mount the ZED to the rover -->
+    Mount the ZED to the rover
     <joint name="zed_front_mount_joint" type="fixed">
         <parent link="base_link"/>
         <child link="zed_front_camera_link"/>
-        <!-- From box geometry: x=0.385-0.065479, y=0, z=0.125+0.217128; 30 deg incline -->
+        From box geometry: x=0.385-0.065479, y=0, z=0.125+0.217128; 30 deg incline
         <origin xyz="0.319521 0.0 0.342128" rpy="0 -0.523599 0"/>
     </joint>
+ -->
     <!-- Additional side cameras -->
     <xacro:zed_camera name="zed_left" model="$(arg camera_model_left)">
