Commit message: Add old point_nav program and update with new options while excluding ekf, turn first then move behaviour turn off wheel and multi camera options in newer point_nav program

File: point_nav/urdf/robot_description.urdf.xacro (robot description, xacro)
@@ -52,5 +52,5 @@
         <material>Gazebo/Blue</material>
     </gazebo>
-    <!-- ZED 2i camera instance (minimal)
+    <!-- ZED 2i camera instance (minimal) -->
     <xacro:zed_camera name="zed_front" model="$(arg camera_model_front)">
         Required block to avoid "Not enough blocks"
@@ -64,6 +64,5 @@
         <origin xyz="0.319521 0.0 0.342128" rpy="0 -0.523599 0"/>
     </joint>
- -->
-    <!-- Additional side cameras -->
+    <!-- Additional side cameras
     <xacro:zed_camera name="zed_left" model="$(arg camera_model_left)">
         <gnss_origin />
@@ -81,5 +80,5 @@
         <child link="zed_right_camera_link"/>
         <origin xyz="0.3095 -0.30232 0.21478" rpy="0 -0.523599 -1.5708"/>
-    </joint>
+    </joint> -->
     <!-- Front Left Wheel Link -->
     <joint name="front_left_wheel_joint" type="continuous">
